Commit message: add gripper config

File: ur10e_gripper_moveit_config/gripper_description/urdf/gripper_macro.xacro (robot description, xacro)
@@ -31,16 +31,10 @@
         </link>
         <!-- TCP frames -->
-        <joint name="${prefix}depth_camera_joint" type="fixed">
-            <origin xyz="0.111986021427 6.69550452272e-8 2.22519248532e-02" rpy="-1.675516081915675 1.6790457912918555e-12 -1.570796326781967" />
-            <parent link="${prefix}end_effector" />
-            <child link="${prefix}depth_camera_tcp" />
-        </joint>
-        <link name="${prefix}depth_camera_tcp" />
-        <joint name="${prefix}rgb_camera_joint" type="fixed">
+        <joint name="${prefix}gripper_joint" type="fixed">
             <origin xyz="0.10554133441 -3.19999999972e-02 1.94659300526e-02" rpy="-1.5707963267928968 0.0 -1.5707963267808966" />
             <parent link="${prefix}end_effector" />
-            <child link="${prefix}rgb_camera_tcp" />
+            <child link="${prefix}gripper_tcp" />
         </joint>
-        <link name="${prefix}rgb_camera_tcp" />
+        <link name="${prefix}gripper_tcp" />
     </xacro:macro>
 </robot>

File: ur10e_gripper_moveit_config/gripper_description/urdf/ur10e_gripper.xacro (robot description, xacro)
@@ -1,4 +1,4 @@
 <?xml version="1.0"?>
-<robot xmlns:xacro="http://wiki.ros.org/xacro" name="ur10e_ka_robot">
+<robot xmlns:xacro="http://wiki.ros.org/xacro" name="ur10e_gripper_robot">
   <!--
     This is a convenience top-level xacro which loads the macro for the UR10

File: ur10e_gripper_moveit_config/gripper_description/urdf/ur10e_gripper_macro.xacro (robot description, xacro)
@@ -17,5 +17,5 @@
           real robot.
   -->
-  <xacro:macro name="ur10e_ka_robot" params="
+  <xacro:macro name="ur10e_gripper_robot" params="
    prefix
    joint_limits_parameters_file:='$(find ur_description)/config/ur10e/joint_limits.yaml'

Commit message: add gripper config

File: ur10e_gripper_moveit_config/gripper_description/urdf/gripper_macro.xacro (robot description, xacro)
@@ -32,5 +32,5 @@
         <!-- TCP frames -->
         <joint name="${prefix}gripper_joint" type="fixed">
-            <origin xyz="0.10554133441 -3.19999999972e-02 1.94659300526e-02" rpy="-1.5707963267928968 0.0 -1.5707963267808966" />
+            <origin xyz="0.116561 2.54033e-08 0.0404998" rpy="-1.5707963267928968 0.0 -1.5707963267808966" />
             <parent link="${prefix}end_effector" />
             <child link="${prefix}gripper_tcp" />

Commit message: gripper example updated

File: ur10e_gripper_moveit_config/gripper_description/urdf/gripper_macro.xacro (robot description, xacro)
@@ -32,5 +32,5 @@
         <!-- TCP frames -->
         <joint name="${prefix}gripper_joint" type="fixed">
-            <origin xyz="0.116561 2.54033e-08 0.0404998" rpy="-1.5707963267928968 0.0 -1.5707963267808966" />
+            <origin xyz="0.03463 -0.05818 0.12491" rpy="-1.5707963267928968 0.0 -2.03156203267928968" />
             <parent link="${prefix}end_effector" />
             <child link="${prefix}gripper_tcp" />
